File: kicad_files/PANEL-COMPLETE.kicad_pcb (KiCad board)
At the start: 2 copper layers, 130 x 190 mm, 287 parts, among them IC1 TPS73533DRBR, IC2 TPS73533DRBR, IC3 TPS73533DRBR, J1 5051101592, J10 5051101592, J11 5051101592, J12 5051101592, J13 5051101592, J2 5051101592, J3 5051101592, J4 5051101592, J5 5051101592, J6 GTFH08131YHR, J7 Conn_01x06, J8 5051101592, J9 Conn_01x02, Q1 TEMT6000X01, Q2 TEMT6000X01, Q3 TEMT6000X01, Q4 BSS138, Q5 TEMT6000X01, Q6 AO3401A, Q7 TEMT6000X01, Q8 Q_NMOS_DGS, SW1 SW_DPST, SW4 SW_SPDT, SW5 SW_SPDT, U1 ATSAMD21G-A, U10 RFM98PW, U11 MCP3427-xUN, U12 BQ25570, U13 MCP3427-xUN, U14 BQ25570, U15 MCP3427-xUN, U16 BQ25570, U17 MCP3427-xUN, U18 BQ25570, U2 MT3608, U4 505110-0697, U5 MPU-9250, U6 MCP73831, U7 MCP3427-xUN, U9 505110-0697, Y1 32.768kHz

Commit message: update components values
Parts:
- C27, C46: value C_Small -> 22uF
- D14: value D_Schottky_Small -> SS34
- L6: value L_Small -> 22uH
- R2, R3, R30, R73, R74, R75, R77, R78, R79, R80, R81, R82: value R_Small -> 10k
- R20, R22, R26: value R -> 1k
- R27: value R_Small -> 110k
- R32: value R_Small -> 1R
- R51, R52, R61, R62, R71, R72: value R_Small -> NOPOP
- R83: value R_Small -> 15k
Changed lines of the file:
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@@
       (effects (font (size 0.75 0.75) (thickness 0.125)))
     )
-    (fp_text value "R_Small" (at 5.08 2.37 90) (layer "F.Fab")
+    (fp_text value "1R" (at 5.08 2.37 90) (layer "F.Fab")
       (effects (font (size 1 1) (thickness 0.15)))
     )
@@
       (effects (font (size 0.75 0.75) (thickness 0.125)))
     )
-    (fp_text value "R_Small" (at 0 1.43) (layer "F.Fab")
+    (fp_text value "10k" (at 0 1.43) (layer "F.Fab")
       (effects (font (size 1 1) (thickness 0.15)))
     )
@@
       (effects (font (size 0.75 0.75) (thickness 0.125)))
     )
-    (fp_text value "R_Small" (at 0 1.43 90) (layer "F.Fab")
+    (fp_text value "10k" (at 0 1.43 90) (layer "F.Fab")
       (effects (font (size 1 1) (thickness 0.15)))
     )
@@
       (effects (font (size 0.75 0.75) (thickness 0.125)))
     )
-    (fp_text value "R_Small" (at 0 1.43) (layer "F.Fab")
+    (fp_text value "10k" (at 0 1.43) (layer "F.Fab")
       (effects (font (size 1 1) (thickness 0.15)))
     )
@@
       (effects (font (size 0.75 0.75) (thickness 0.125)) (justify mirror))
     )
-    (fp_text value "R_Small" (at 0 -1.43) (layer "B.Fab")
+    (fp_text value "10k" (at 0 -1.43) (layer "B.Fab")
       (effects (font (size 1 1) (thickness 0.15)) (justify mirror))
     )
@@
       (effects (font (size 0.75 0.75) (thickness 0.125)) (justify mirror))
     )
-    (fp_text value "R_Small" (at 0 -1.17 90) (layer "B.Fab")
+    (fp_text value "NOPOP" (at 0 -1.17 90) (layer "B.Fab")
       (effects (font (size 1 1) (thickness 0.15)) (justify mirror))
     )
@@
       (effects (font (size 1 1) (thickness 0.15)))
     )
-    (fp_text value "C_Small" (at 0 -1.85) (layer "B.Fab")
+    (fp_text value "22uF" (at 0 -1.85) (layer "B.Fab")
       (effects (font (size 1 1) (thickness 0.15)) (justify mirror))
     )
@@
       (effects (font (size 0.75 0.75) (thickness 0.125)) (justify mirror))
     )
-    (fp_text value "R_Small" (at 0 -1.17) (layer "B.Fab")
+    (fp_text value "NOPOP" (at 0 -1.17) (layer "B.Fab")
       (effects (font (size 1 1) (thickness 0.15)) (justify mirror))
     )
@@
       (effects (font (size 1 1) (thickness 0.15)) (justify mirror))
     )
-    (fp_text value "C_Small" (at 0 -1.85 90) (layer "B.Fab")
+    (fp_text value "22uF" (at 0 -1.85 90) (layer "B.Fab")
       (effects (font (size 1 1) (thickness 0.15)) (justify mirror))
     )
@@
       (effects (font (size 1 1) (thickness 0.15)) (justify mirror))
     )
-    (fp_text value "R_Small" (at 0 -1.43 90) (layer "B.Fab")
+    (fp_text value "110k" (at 0 -1.43 90) (layer "B.Fab")
       (effects (font (size 1 1) (thickness 0.15)) (justify mirror))
     )
@@
       (effects (font (size 0.75 0.75) (thickness 0.125)) (justify mirror))
     )
-    (fp_text value "R_Small" (at 0 -1.43) (layer "B.Fab")
+    (fp_text value "10k" (at 0 -1.43) (layer "B.Fab")
       (effects (font (size 1 1) (thickness 0.15)) (justify mirror))
     )
@@
       (effects (font (size 0.75 0.75) (thickness 0.125)) (justify mirror))
     )
-    (fp_text value "R_Small" (at 0 -1.17 90) (layer "B.Fab")
+    (fp_text value "NOPOP" (at 0 -1.17 90) (layer "B.Fab")
       (effects (font (size 1 1) (thickness 0.15)) (justify mirror))
     )
@@
       (effects (font (size 1 1) (thickness 0.15)) (justify mirror))
     )
-    (fp_text value "R_Small" (at 0 -1.43 90) (layer "B.Fab")
+    (fp_text value "15k" (at 0 -1.43 90) (layer "B.Fab")
       (effects (font (size 1 1) (thickness 0.15)) (justify mirror))
     )
@@
       (effects (font (size 0.75 0.75) (thickness 0.125)) (justify mirror))
     )
-    (fp_text value "R_Small" (at 0 -1.17 90) (layer "B.Fab")
+    (fp_text value "10k" (at 0 -1.17 90) (layer "B.Fab")
       (effects (font (size 1 1) (thickness 0.15)) (justify mirror))
     )
@@
       (effects (font (size 0.75 0.75) (thickness 0.125)) (justify mirror))
     )
-    (fp_text value "R_Small" (at 0 -1.17) (layer "B.Fab")
+    (fp_text value "NOPOP" (at 0 -1.17) (layer "B.Fab")
       (effects (font (size 1 1) (thickness 0.15)) (justify mirror))
     )
@@
       (effects (font (size 1 1) (thickness 0.15)))
     )
-    (fp_text value "R" (at 0 -1.43) (layer "B.Fab")
+    (fp_text value "1k" (at 0 -1.43) (layer "B.Fab")
       (effects (font (size 1 1) (thickness 0.15)) (justify mirror))
     )
@@
       (effects (font (size 0.75 0.75) (thickness 0.125)) (justify mirror))
     )
-    (fp_text value "R_Small" (at 0 -1.43 90) (layer "B.Fab")
+    (fp_text value "10k" (at 0 -1.43 90) (layer "B.Fab")
       (effects (font (size 1 1) (thickness 0.15)) (justify mirror))
     )
@@
       (effects (font (size 0.75 0.75) (thickness 0.125)) (justify mirror))
     )
-    (fp_text value "R_Small" (at 0 -1.43) (layer "B.Fab")
+    (fp_text value "10k" (at 0 -1.43) (layer "B.Fab")
       (effects (font (size 1 1) (thickness 0.15)) (justify mirror))
     )
@@
       (effects (font (size 1 1) (thickness 0.15)))
     )
-    (fp_text value "R" (at 0 -1.43) (layer "B.Fab")
+    (fp_text value "1k" (at 0 -1.43) (layer "B.Fab")
       (effects (font (size 1 1) (thickness 0.15)) (justify mirror))
     )
@@
       (effects (font (size 1 1) (thickness 0.15)) (justify mirror))
     )
-    (fp_text value "D_Schottky_Small" (at 0 -2.6 90) (layer "B.Fab")
+    (fp_text value "SS34" (at 0 -2.6 90) (layer "B.Fab")
       (effects (font (size 1 1) (thickness 0.15)) (justify mirror))
     )
@@
       (effects (font (size 1 1) (thickness 0.15)))
     )
-    (fp_text value "R" (at 0 -1.43) (layer "B.Fab")
+    (fp_text value "1k" (at 0 -1.43) (layer "B.Fab")
       (effects (font (size 1 1) (thickness 0.15)) (justify mirror))
     )
@@
       (effects (font (size 0.75 0.75) (thickness 0.125)) (justify mirror))
     )
-    (fp_text value "R_Small" (at 0 -1.43 90) (layer "B.Fab")
+    (fp_text value "10k" (at 0 -1.43 90) (layer "B.Fab")
       (effects (font (size 1 1) (thickness 0.15)) (justify mirror))
     )
@@
       (effects (font (size 0.75 0.75) (thickness 0.125)) (justify mirror))
     )
-    (fp_text value "R_Small" (at 0 -1.17 90) (layer "B.Fab")
+    (fp_text value "NOPOP" (at 0 -1.17 90) (layer "B.Fab")
       (effects (font (size 1 1) (thickness 0.15)) (justify mirror))
     )
@@
       (effects (font (size 0.75 0.75) (thickness 0.125)) (justify mirror))
     )
-    (fp_text value "R_Small" (at 0 -1.43 90) (layer "B.Fab")
+    (fp_text value "10k" (at 0 -1.43 90) (layer "B.Fab")
       (effects (font (size 1 1) (thickness 0.15)) (justify mirror))
     )
@@
       (effects (font (size 0.75 0.75) (thickness 0.125)) (justify mirror))
     )
-    (fp_text value "R_Small" (at 0 -1.43) (layer "B.Fab")
+    (fp_text value "10k" (at 0 -1.43) (layer "B.Fab")
       (effects (font (size 1 1) (thickness 0.15)) (justify mirror))
     )
@@
       (effects (font (size 0.75 0.75) (thickness 0.125)) (justify mirror))
     )
-    (fp_text value "R_Small" (at 0 -1.17 90) (layer "B.Fab")
+    (fp_text value "NOPOP" (at 0 -1.17 90) (layer "B.Fab")
       (effects (font (size 1 1) (thickness 0.15)) (justify mirror))
     )
@@
       (effects (font (size 1 1) (thickness 0.15)) (justify mirror))
     )
-    (fp_text value "L_Small" (at 0 -4.45) (layer "B.Fab")
+    (fp_text value "22uH" (at 0 -4.45) (layer "B.Fab")
       (effects (font (size 1 1) (thickness 0.15)) (justify mirror))
     )
@@
       (effects (font (size 0.75 0.75) (thickness 0.125)) (justify mirror))
     )
-    (fp_text value "R_Small" (at 0 -1.43 90) (layer "B.Fab")
+    (fp_text value "10k" (at 0 -1.43 90) (layer "B.Fab")
       (effects (font (size 1 1) (thickness 0.15)) (justify mirror))
     )
