File: kicad_files/obdh.kicad_sch (KiCad schematic)
At the start: 97 parts, among them IC1 TPS73533DRBR, IC2 TPS73533DRBR, IC3 TPS73533DRBR, J1 5051101592, J2 5051101592, J3 5051101592, J4 5051101592, J5 5051101592, J6 GTFH08131YHR, J7 Conn_01x06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

Commit message: update components values
Parts:
- C27, C46: value C_Small -> 22uF
- D14: value D_Schottky_Small -> SS34
- L6: value L_Small -> 22uH
- R2, R3, R75: value R_Small -> 10k
- R20, R22, R26: value R -> 1k
- R27: value R_Small -> 110k
- R83: value R_Small -> 15k
Changed lines of the file:
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@@
   (symbol (lib_id "Device:L_Small") (at 405.13 99.695 90) (unit 1)
     (in_bom yes) (on_board yes) (fields_autoplaced)
-    (property "Reference" "L6" (id 0) (at 405.13 94.615 90))
-    (property "Value" "L_Small" (id 1) (at 405.13 97.155 90))
+    (property "Reference" "L6" (id 0) (at 405.13 93.98 90))
+    (property "Value" "22uH" (id 1) (at 405.13 96.52 90))
     (property "Footprint" "Inductor_SMD:L_6.3x6.3_H3" (id 2) (at 405.13 99.695 0)
       (effects (font (size 1.27 1.27)) hide)
@@
   (symbol (lib_id "Device:R_Small") (at 422.91 118.11 0) (unit 1)
     (in_bom yes) (on_board yes) (fields_autoplaced)
-    (property "Reference" "R83" (id 0) (at 424.815 116.8399 0)
-      (effects (font (size 1.27 1.27)) (justify left))
-    )
-    (property "Value" "R_Small" (id 1) (at 424.815 119.3799 0)
+    (property "Reference" "R83" (id 0) (at 425.45 116.8399 0)
+      (effects (font (size 1.27 1.27)) (justify left))
+    )
+    (property "Value" "15k" (id 1) (at 425.45 119.3799 0)
       (effects (font (size 1.27 1.27)) (justify left))
     )
@@
   (symbol (lib_id "Device:D_Schottky_Small") (at 418.465 106.68 180) (unit 1)
     (in_bom yes) (on_board yes) (fields_autoplaced)
-    (property "Reference" "D14" (id 0) (at 418.719 100.965 0))
-    (property "Value" "D_Schottky_Small" (id 1) (at 418.719 103.505 0))
+    (property "Reference" "D14" (id 0) (at 418.719 100.33 0))
+    (property "Value" "SS34" (id 1) (at 418.719 102.87 0))
     (property "Footprint" "Diode_SMD:D_SMA" (id 2) (at 418.465 106.68 90)
       (effects (font (size 1.27 1.27)) hide)
@@
       (effects (font (size 1.27 1.27)) (justify left))
     )
-    (property "Value" "R_Small" (id 1) (at 68.58 351.7899 0)
+    (property "Value" "10k" (id 1) (at 68.58 351.7899 0)
       (effects (font (size 1.27 1.27)) (justify left))
     )
@@
   )
   (symbol (lib_id "Device:R_Small") (at 274.955 104.775 0) (mirror x) (unit 1)
-    (in_bom yes) (on_board yes) (fields_autoplaced)
-    (property "Reference" "R75" (id 0) (at 272.415 103.5049 0)
-      (effects (font (size 1.27 1.27)) (justify right))
-    )
-    (property "Value" "R_Small" (id 1) (at 272.415 106.0449 0)
+    (in_bom yes) (on_board yes)
+    (property "Reference" "R75" (id 0) (at 273.05 103.5049 0)
+      (effects (font (size 1.27 1.27)) (justify right))
+    )
+    (property "Value" "10k" (id 1) (at 273.05 106.0449 0)
       (effects (font (size 1.27 1.27)) (justify right))
     )
@@
       (effects (font (size 1.27 1.27)) (justify left))
     )
-    (property "Value" "R_Small" (id 1) (at 425.45 111.7599 0)
+    (property "Value" "110k" (id 1) (at 425.45 111.7599 0)
       (effects (font (size 1.27 1.27)) (justify left))
     )
@@
       (effects (font (size 1.27 1.27)) (justify left))
     )
-    (property "Value" "R_Small" (id 1) (at 68.58 361.3149 0)
+    (property "Value" "10k" (id 1) (at 68.58 361.3149 0)
       (effects (font (size 1.27 1.27)) (justify left))
     )
@@
       (effects (font (size 1.27 1.27)) (justify left))
     )
-    (property "Value" "R" (id 1) (at 242.57 355.6 0)
+    (property "Value" "1k" (id 1) (at 242.57 355.6 0)
       (effects (font (size 1.27 1.27)) (justify left))
     )
@@
       (effects (font (size 1.27 1.27)) (justify left))
     )
-    (property "Value" "R" (id 1) (at 259.08 355.6 0)
+    (property "Value" "1k" (id 1) (at 259.08 355.6 0)
       (effects (font (size 1.27 1.27)) (justify left))
     )
@@
   (symbol (lib_id "Device:C_Small") (at 384.81 116.205 0) (mirror x) (unit 1)
     (in_bom yes) (on_board yes) (fields_autoplaced)
-    (property "Reference" "C27" (id 0) (at 381.635 114.9285 0)
-      (effects (font (size 1.27 1.27)) (justify right))
-    )
-    (property "Value" "C_Small" (id 1) (at 381.635 117.4685 0)
+    (property "Reference" "C27" (id 0) (at 382.27 114.9285 0)
+      (effects (font (size 1.27 1.27)) (justify right))
+    )
+    (property "Value" "22uF" (id 1) (at 382.27 117.4685 0)
       (effects (font (size 1.27 1.27)) (justify right))
     )
@@
       (effects (font (size 1.27 1.27)) (justify left))
     )
-    (property "Value" "R" (id 1) (at 227.33 355.6 0)
+    (property "Value" "1k" (id 1) (at 227.33 355.6 0)
       (effects (font (size 1.27 1.27)) (justify left))
     )
@@
       (effects (font (size 1.27 1.27)) (justify left))
     )
-    (property "Value" "C_Small" (id 1) (at 439.42 115.5762 0)
-      (effects (font (size 1.27 1.27)) (justify left))
-    )
+    (property "Value" "22uF" (id 1) (at 439.42 115.5762 0)
+      (effects (font (size 1.27 1.27)) (justify left))
+    )
